File: hardware/Nixie_RevC_placement.kicad_pcb (KiCad board)
At the start: 4 copper layers, 218 x 64 mm, 80 parts, among them J1 12 V pigtail pads, J2 CR2032 lead pads, SW1 B3F-1062-G (SET), SW2 B3F-1062-G (H), SW3 B3F-1062-G (M), T1 IN-14, T2 IN-14, T3 IN-14, T4 IN-14, T5 IN-14, T6 IN-14, U1 HV5522PJ-G, U2 HV5522PJ-G, U3 DS3231SN#

Commit message: Six-Tube Nixie Clock Rev C: alarm-clock case, build guide, KiCad, CAD, firmware, website and desktop app
Parts:
- JP1, TP1, TP2, TP3, TP4: moved to F.Cu
- moved TP1 80.1 mm to (120.0, 32.0)
- moved TP4 39.3 mm to (126.0, 32.0)
- moved JP1 16.6 mm to (110.0, 34.0)
- moved TP2 5.66 mm to (200.0, 32.0)
- moved TP3 4.47 mm to (206.0, 32.0)
